Commit message: Make URDF mesh paths portable (package:// not absolute)
The generated URDF had absolute /Users/samarthmahapatra/... paths baked
into every <mesh filename>, so it only loaded on the machine it was
generated on. Rewrite them to package://abb_crb15000_support/... so the
_resolve_mesh handler resolves them relative to the repo's abb_desc/ on
any machine.

Co-Authored-By: Claude Opus 4.8 (1M context) <noreply@anthropic.com>

File: crb15000_12_127.urdf (robot description, URDF)
Before this commit: robot abb_crb15000_12_127, 10 links, 9 joints
Links:
- link base_link: geometry collision mesh filename=package://abb_crb15000_support/meshes/crb15000_12_127/colli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; visual mesh filename=package://abb_crb15000_support/meshes/crb15000_12_127/visua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
- link link_1: geometry collision mesh filename=package://abb_crb15000_support/meshes/crb15000_12_127/colli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; visual mesh filename=package://abb_crb15000_support/meshes/crb15000_12_127/visua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
- link link_2: geometry collision mesh filename=package://abb_crb15000_support/meshes/crb15000_12_127/colli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; visual mesh filename=package://abb_crb15000_support/meshes/crb15000_12_127/visua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
- link link_3: geometry collision mesh filename=package://abb_crb15000_support/meshes/crb15000_5_95/collisi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; visual mesh filename=package://abb_crb15000_support/meshes/crb15000_5_95/visual/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
- link link_4: geometry collision mesh filename=package://abb_crb15000_support/meshes/crb15000_12_127/colli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; visual mesh filename=package://abb_crb15000_support/meshes/crb15000_12_127/visua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
- link link_5: geometry collision mesh filename=package://abb_crb15000_support/meshes/crb15000_5_95/collisi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; visual mesh filename=package://abb_crb15000_support/meshes/crb15000_5_95/visual/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
- link link_6: geometry collision mesh filename=package://abb_crb15000_support/meshes/crb15000_5_95/collisi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; visual mesh filename=package://abb_crb15000_support/meshes/crb15000_5_95/visual/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
